File: KiCad_perfboard_sketch/ra_perfboard/ra_perfboard.kicad_sch (KiCad schematic)
At the start: 20 parts, among them J1 M1, J10 L6, J2 M2, J3 Terminal, J4 USART, J5 L3, J6 L1, J7 L2, J8 L4, J9 L5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

Commit message: Final commit after submitting project. Currently no plans to proegress in this project any further.
Parts:
- added C5: M3_Cap, Capacitor_THT:CP_Radial_D5.0mm_P2.50mm, symbol Device:C_Polarized
- added C6, C8: 100nF, Capacitor_THT:C_Disc_D3.0mm_W2.0mm_P2.50mm, symbol Device:C
- added C7: M4_Cap, Capacitor_THT:CP_Radial_D5.0mm_P2.50mm, symbol Device:C_Polarized
- added J11: M3, Connector_PinHeader_2.54mm:PinHeader_1x04_P2.54mm_Vertical, symbol Connector:Conn_01x04_Pin
- added J12: M4, Connector_PinHeader_2.54mm:PinHeader_1x04_P2.54mm_Vertical, symbol Connector:Conn_01x04_Pin
- added U6, U7: ~, stm32_ra_board_footprints:TMC2208_Board_Footprint, symbol stm32_ra_boards:TMC2208
Connections:
- net +24V: now also C5.1, C7.1, U6.16 (+VMOT), U7.16 (+VMOT)
- net +3V3: now also C6.1, C8.1, U6.10 (VIO), U6.2 (MS1), U6.3 (MS2), U7.10 (VIO), U7.2 (MS1), U7.3 (MS2)
- net GND: now also C5.2, C6.2, C7.2, C8.2, U6.15 (GND), U6.9 (GND), U7.15 (GND), U7.9 (GND)
- net M3_EN: now reaches U4.10 (PA4)
- net M3_EN: now also U6.1 (EN)
- net M3_DIR: now reaches U4.11 (PA5)
- net M3_DIR: now also U6.8 (DIR)
- net M3_STEP: now reaches U4.12 (PA6)
- net M3_STEP: now also U6.7 (STEP)
- net M4_DIR: now reaches U4.31 (PA15)
- net M4_DIR: now also U7.8 (DIR)
- net M4_EN: now reaches U4.32 (PA12)
- net M4_EN: now also U7.1 (EN), U7.7 (STEP)
- net M4_STEP: now reaches U4.33 (PA11)
- new net: J12.1 (Pin_1), U7.11 (1B)
- new net: J12.2 (Pin_2), U7.12 (1A)
- new net: J12.3 (Pin_3), U7.13 (2A)
- new net: J12.4 (Pin_4), U7.14 (2B)
- new net: J11.1 (Pin_1), U6.11 (1B)
- new net: J11.2 (Pin_2), U6.12 (1A)
- new net: J11.3 (Pin_3), U6.13 (2A)
- new net: J11.4 (Pin_4), U6.14 (2B)
- no-connect marks 38 -> 41
Other:
- note added: "FTDI HEADERS"
- note added: "SENSOR HEADERS"
- note removed: "SENSOR AND FTDI HEADERS"
- title: (none) -> Robot Arm Circuit
- moved on the sheet: C1, C2, C3, C4, D1, J1, J10, J2, J3, J4, J5, J6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
